File: Spin_Coater_Circuit/Design_File/Spct.kicad_sch (KiCad schematic)
At the start: 42 parts, among them J1 Conn_01x02_Pin, J2 Conn_01x03_Pin, J3 Conn_01x08_Pin, J4 Conn_01x02_Pin, J5 Conn_01x04_Pin, J6 Conn_01x02_Pin, J7 Conn_01x06_Pin, J8 Conn_01x02_Pin, J9 Conn_01x02_Pin, Q1 PNP, Q2 PNP, Q3 PNP, U1 NUCLEO-F401RE, U2 MCP4922-EP, U4 24LC512

Commit message: Change Ver1.1
Parts:
- removed Q1: PNP, Package_TO_SOT_THT:TO-92, symbol Simulation_SPICE:PNP
- added D5: Zener_6V, Diode_THT:D_5W_P12.70mm_Horizontal, symbol Device:D_Zener
- BZ1: value Buzzer -> IMT12D2001AP-Buzzer
- C2, C3: footprint Capacitor_THT:C_Disc_D3.4mm_W2.1mm_P2.50mm -> Capacitor_THT:C_Disc_D4.3mm_W1.9mm_P5.00mm
- D1: value Zener_12V -> Zener_6V; footprint Diode_THT:D_5W_P10.16mm_Horizontal -> Diode_THT:D_5W_P12.70mm_Horizontal
- Q2, Q3: value PNP -> NPN; footprint Package_TO_SOT_THT:TO-92 -> Package_TO_SOT_THT:TO-92L_Inline_Wide_ECB; symbol Simulation_SPICE:PNP -> Simulation_SPICE:NPN
- R1: value 330 -> 100; footprint Resistor_THT:R_Axial_DIN0204_L3.6mm_D1.6mm_P5.08mm_Horizontal -> Resistor_THT:R_Axial_DIN0207_L6.3mm_D2.5mm_P10.16mm_Horizontal
- R10, R11, R12, R13, R14, R16, R17, R18, R2, R3, R4, R5, R6, R8, R9: footprint Resistor_THT:R_Axial_DIN0204_L3.6mm_D1.6mm_P5.08mm_Horizontal -> Resistor_THT:R_Axial_DIN0207_L6.3mm_D2.5mm_P10.16mm_Horizontal
- R7: value 10k -> 100; footprint Resistor_THT:R_Axial_DIN0204_L3.6mm_D1.6mm_P5.08mm_Horizontal -> Resistor_THT:R_Axial_DIN0207_L6.3mm_D2.5mm_P10.16mm_Horizontal
- U1: footprint ST_NUCLEO-F401RE -> Module:ST_NUCLEO-F401RE
- U3: value ~ -> 367661
Connections:
- net +12V: now also D5.2 (A); no longer D1.2 (A)
- net +3V3: no longer R11.2
- net EMO: now also Q2.3 (B); no longer Q2.2 (B)
- net Lid_Sensor: now also Q3.3 (B); no longer Q3.2 (B)
- net cRPM_METER: now also R11.1; no longer R4.1
- net at J3.8 (Pin_8), U3.9 (H3): now also R11.2; no longer R11.1
- net READY_IN: now reaches U1.CN7_2 (PC11)
- net READY_IN: now also R5.1, U3.10 (Ready)
- net at R7.2, U3.13 (EN): now also Q2.2 (C), Q3.2 (C); no longer Q2.3 (E), Q3.3 (E)
- net Phase_MON: now reaches U1.CN10_35 (PA2)
- net Phase_MON: now also R4.1
- new net: D1.2 (A), D5.1 (K)
Other:
- note added: "EMR Off -> LOW EMR On -> HIGH"
- note added: "Enable = HIGH Disable = LOW"
- note added: "Magnet O -> HIGH Magnet X -> LOW"
- note added: "Revision History - V 0.1 [-] Change capacitor layout size to large - Change resistor layout size to large [-] Add zener diode to decrease heat - Change BJT layout pinmap - Change PWM reading pin to ADC pin -"
- note removed: "EMR On -> LOW EMR Off -> HIGH"
- note removed: "Magnet O -> LOW Magnet X -> HIGH"
- moved on the sheet: D4, R11, R5

Commit message: Circuit version 1.2
Parts:
- removed D1, D5: Zener_6V, Diode_THT:D_5W_P12.70mm_Horizontal, symbol Device:D_Zener
- added U5: SZH-PWSD-026, Symbol:DCDC_SZH-PWSD-026, symbol Converter_DCDC:SZH-PWSD-026
- Q2, Q3: symbol Simulation_SPICE:NPN -> Simulation_SPICE:NMOS
Connections:
- net +12V: now also U5.1 (VOUT), U5.2 (VOUT)
- net +24V: now also C2.1, J3.5 (Pin_5), U3.6 (HALL_5V), U5.7 (VIN), U5.8 (VIN)
- net EMO: now also Q2.2 (G); no longer Q2.3 (B)
- net GND: now also Q2.3 (S), Q3.3 (S), U5.3 (GND), U5.4 (GND), U5.5 (GND), U5.6 (GND); no longer Q2.1 (E), Q3.1 (E)
- net Lid_Sensor: now also Q3.2 (G); no longer Q3.3 (B)
- net at R7.2, U3.13 (EN): now also Q2.1 (D), Q3.1 (D); no longer Q2.2 (C), Q3.2 (C)
Other:
- note added: "Revision History - V 1.1 [-] Change capacitor layout size to large [-] Change resistor layout size to large [-] Add zener diode to decrease heat [-] Change BJT layout pinmap [-] Change PWM reading pin to ADC pin - V 1.2 [ ] Change NPN to N-FET mosfet. [ ] Zener Diode to DC/DC Converter [ ] BEMF Block"
- note removed: "Revision History - V 0.1 [-] Change capacitor layout size to large - Change resistor layout size to large [-] Add zener diode to decrease heat - Change BJT layout pinmap - Change PWM reading pin to ADC pin -"

Commit message: Spin coater ver1.3
Parts:
- removed BZ1: IMT12D2001AP-Buzzer, Buzzer_Beeper:MagneticBuzzer_ProSignal_ABT-410-RC, symbol Device:Buzzer
- removed U5: SZH-PWSD-026, Symbol:DCDC_SZH-PWSD-026, symbol Converter_DCDC:SZH-PWSD-026
- added C10, C11, C15: 10uF/10V, Capacitor_SMD:C_0805_2012Metric, symbol Device:C
- added C12, C4, C6, C7: 100nF/50V, Capacitor_SMD:C_0603_1608Metric, symbol Device:C
- added C13, C14: 22uF/10V, Capacitor_SMD:C_0805_2012Metric, symbol Device:C
- added C5: 4.7F/50V, Capacitor_SMD:C_1206_3216Metric, symbol Device:C
- added C8: 1uF/10V, Capacitor_SMD:C_0603_1608Metric, symbol Device:C
- added C9: 27pF/10V, Capacitor_SMD:C_0603_1608Metric, symbol Device:C
- added D1: B360B-13-F, Diode_SMD:D_SMB, symbol Diode:1N5401
- added L1: 22uH, Custom_Library:L_Bourns_SRR6028, symbol Device:L_Iron_Small
- added LS1: CMT-7525-80-SMT-TR, Custom_Library:XDCR_CMT-7525-80-SMT-TR, symbol Custom_Library:CMT-7525-80-SMT-TR
- added Q1: 2N7002, Package_TO_SOT_SMD:SOT-23, symbol Custom_Library:NMOS
- added R15: 10k, Resistor_SMD:R_0603_1608Metric, symbol Device:R
- added R19, R20, R23: 75k, Resistor_SMD:R_0603_1608Metric, symbol Device:R
- added R21: 0, Resistor_SMD:R_0603_1608Metric, symbol Device:R
- added R22: N.C, Resistor_SMD:R_0603_1608Metric, symbol Device:R
- added U6: ISL85410FRZ, Custom_Library:SON50P300X300X100-13N_270X200_, symbol Custom_Library:ISL85410FRZ
- C1: value 330uF / 50V -> 330uF/50V; footprint Capacitor_THT:CP_Radial_D10.0mm_P5.00mm -> Custom_Library:CP_Elec_12.5x12.5; Manufacturer (none) -> Chemi-con/EMVH500ARA331MKG5S
- C2, C3: value 100nF -> 100nF/50V; footprint Capacitor_THT:C_Disc_D4.3mm_W1.9mm_P5.00mm -> Capacitor_SMD:C_0603_1608Metric; Manufacturer (none) -> Samsung/CL10B104MB8NNNC
- D2: value 1N5401 -> B360B-13-F; footprint Diode_THT:D_DO-201AD_P15.24mm_Horizontal -> Diode_SMD:D_SMB
- D3: value Zener_3.3V -> MM3Z3V3T1G; footprint Diode_THT:D_5W_P10.16mm_Horizontal -> Custom_Library:D_SOD-323-2; Manufacturer (none) -> Onsemni
- D4: value LED -> 150060BS55040; footprint LED_THT:LED_D3.0mm -> LED_SMD:LED_0603_1608Metric; Manufacturer (none) -> Würth Elektronik
- F1: value Fuse_3A -> 0679H5000-01; footprint Fuse:Fuse_Littelfuse-LVR100 -> Custom_Library:Fuse_2410_6225_Metric
- J1, J4, J6, J8, J9: value Conn_01x02_Pin -> EH_B2B-EH-A; Manufacturer (none) -> JST
- J2: value Conn_01x03_Pin -> EH_B3B-EH-A; Manufacturer (none) -> JST
- J3: value Conn_01x08_Pin -> EH_B8B-EH-A; Manufacturer (none) -> JST
- J5: value Conn_01x04_Pin -> EH_B4B-EH-A; Manufacturer (none) -> JST
- J7: value Conn_01x06_Pin -> EH_B6B-EH-A; Manufacturer (none) -> JST
- Q2, Q3: value NPN -> 2N7002; footprint Package_TO_SOT_THT:TO-92L_Inline_Wide_ECB -> Package_TO_SOT_SMD:SOT-23; symbol Simulation_SPICE:NMOS -> Custom_Library:NMOS
- R1, R10, R11, R12, R13, R14, R16, R17, R18, R2, R3, R4, R5, R6, R7, R8, R9: footprint Resistor_THT:R_Axial_DIN0207_L6.3mm_D2.5mm_P10.16mm_Horizontal -> Resistor_SMD:R_0603_1608Metric
- U1: value NUCLEO-F401RE -> NUCLEO-F411RE
- U2: value MCP4922-EP -> MCP4922-E/SL; footprint Package_DIP:DIP-14_W7.62mm_Socket -> Package_SO:SOIC-14_3.9x8.7mm_P1.27mm; Manufacturer (none) -> Microchips
- U4: value 24LC512 -> 24LC512T-I/SN; footprint Package_DIP:DIP-8_W7.62mm_Socket -> Package_SO:SOIC-8_5.275x5.275mm_P1.27mm; Manufacturer (none) -> Microchips
Connections:
- net +24V: now also C5.1, C6.1, R20.1, U6.4 (VIN); no longer C2.1, J3.5 (Pin_5), U3.6 (HALL_5V)
- net +3V3: now also D1.1 (K), LS1.P
- net EMO: now also Q2.1 (G); no longer Q2.2 (G)
- net GND: now also Q2.2 (S), Q3.2 (S), C10.2, C11.2, C12.2, C13.2, C14.2, C15.2, C4.2, C5.2, C6.2, C8.2, Q1.2 (S), R15.2, R22.2, R23.1, U6.13 (EXP), U6.6 (PGND); no longer Q2.3 (S), Q3.3 (S)
- net Lid_Sensor: now also Q3.1 (G), C4.1; no longer Q3.2 (G)
- net +E5V: now reaches U1.CN7_6 (E5V)
- net +E5V: now also C3.1, U2.1 (VDD), U2.11 (VrefB), U2.13 (VrefA), U2.9 (~{SHDN}), C10.1, C11.1, C12.1, C13.1, C14.1, C15.1, C9.1, L1.2, R19.1
- net at R7.2, U3.13 (EN): now also Q2.3 (D), Q3.3 (D); no longer Q2.1 (D), Q3.1 (D)
- net at R12.1: now also Q1.1 (G)
- removed net +5V: C3.1, U1.CN7_18 (+5V_S1), U2.1 (VDD), U2.11 (VrefB), U2.13 (VrefA), U2.9 (~{SHDN})
- new net: D1.2 (A), LS1.N, Q1.3 (D)
- new net: C2.1, J3.5 (Pin_5), U3.6 (HALL_5V)
- new net: R20.2, U6.7 (EN)
- new net: R21.1, R22.1, U6.12 (FS)
- new net: C9.2, R15.1, R19.2, U6.10 (FB)
- new net: R23.2, U6.2 (SYNC)
- new net: C7.1, U6.3 (BOOT)
- new net: C7.2, L1.1, U6.5 (PHASE)
- new net: C8.1, R21.2, U6.1 (SS), U6.11 (COMP), U6.9 (VCC)
Other:
- note added: "3-40V"
- note added: "5.1V"
- note added: "Address - b1010000"
- note added: "Revision History - V 1.1 [-] Change capacitor layout size to large [-] Change resistor layout size to large [-] Add zener diode to decrease heat [-] Change BJT layout pinmap [-] Change PWM reading pin to ADC pin - V 1.2 [ ] Change NPN to N-FET mosfet. [ ] Zener Diode to DC/DC Converter [ ] BEMF Block - V 1.3 [-] Change R,C,D size to SMD [-] Embedded DC/DC"
- note removed: "Revision History - V 1.1 [-] Change capacitor layout size to large [-] Change resistor layout size to large [-] Add zener diode to decrease heat [-] Change BJT layout pinmap [-] Change PWM reading pin to ADC pin - V 1.2 [ ] Change NPN to N-FET mosfet. [ ] Zener Diode to DC/DC Converter [ ] BEMF Block"
- moved on the sheet: C1, C2, D2, D3, D4, F1, J1, J2, J3, J5, Q2, Q3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

Commit message: version 2.0 circuit init
Parts:
- removed J4, J6, J8, J9: EH_B2B-EH-A, Connector_JST:JST_EH_B2B-EH-A_1x02_P2.50mm_Vertical, symbol Connector:Conn_01x02_Pin
- removed J7: EH_B6B-EH-A, Connector_JST:JST_EH_B6B-EH-A_1x06_P2.50mm_Vertical, symbol Connector:Conn_01x06_Pin
- removed R14, R8: 10k, Resistor_SMD:R_0603_1608Metric, symbol Device:R
- added D5: NSR20F30NXT5G, Custom_Library:DSN2-152AB_ONS, symbol Custom_Library:NSR20F30NXT5G
- added J10: Conn_01x08, Connector_PinHeader_2.54mm:PinHeader_1x08_P2.54mm_Vertical, symbol Connector_Generic:Conn_01x08
- added J11: Conn_02x09_Odd_Even, Connector_PinHeader_2.54mm:PinHeader_2x09_P2.54mm_Vertical, symbol Connector_Generic:Conn_02x09_Odd_Even
- added J12: Motor_Output, Connector_Molex:Molex_Mini-Fit_Jr_5569-04A2_2x02_P4.20mm_Horizontal, symbol Connector_Generic:Conn_02x02_Counter_Clockwise
- added J13: Motor_Feedback, Connector_Molex:Molex_Micro-Fit_3.0_43045-0621_2x03-1MP_P3.00mm_Horizontal, symbol Connector_Generic:Conn_02x03_Counter_Clockwise
- added J14: Conn_01x10, symbol Connector_Generic:Conn_01x10
- added J15, J16: Conn_01x08, symbol Connector_Generic:Conn_01x08
- added J17: Conn_01x06, symbol Connector_Generic:Conn_01x06
- added J18: USB_C_Receptacle_USB2.0_14P, Connector_USB:USB_C_Receptacle_G-Switch_GT-USB-7010ASV, symbol Connector:USB_C_Receptacle_USB2.0_14P
- added R24: 100, Resistor_SMD:R_0603_1608Metric, symbol Device:R
- added R25: 100k, Resistor_SMD:R_0603_1608Metric, symbol Device:R
- added U5: STM32F411RETx, Package_QFP:LQFP-64_10x10mm_P0.5mm, symbol MCU_ST_STM32F4:STM32F411RETx
- added U7: FT231XQ, Package_DFN_QFN:QFN-20-1EP_4x4mm_P0.5mm_EP2.5x2.5mm, symbol Interface_USB:FT231XQ
- added U8: ADPL42005ACPZ-3.3-R7, Package_CSP:LFCSP-8-1EP_3x3mm_P0.5mm_EP1.6x2.34mm, symbol Custom_Library:ADPL42005ACPZ-3.3-R7
Connections:
- net +24V: now also J11.7 (Pin_7), J11.8 (Pin_8)
- net +3V3: now also J16.4 (Pin_4), U5.13 (VDDA), U5.19 (VDD), U5.32 (VDD), U5.48 (VDD), U5.64 (VDD), U8.1 (VOUT), U8.2 (SENSE)
- net +E5V: now also D5.1 (K), U8.5 (EN), U8.8 (VIN)
- net ADC_UPDATE: now also U5.35 (PB14)
- net DIR: now also U5.24 (PC4); no longer U1.CN7_1 (PC10)
- net DRV_EN: now also U5.27 (PB1); no longer U1.CN7_3 (PC12)
- net EMO: no longer U1.CN7_25 (PC14)
- net GND: now also J10.6 (Pin_6), J11.10 (Pin_10), J11.14 (Pin_14), J11.16 (Pin_16), J11.18 (Pin_18), J11.9 (Pin_9), J13.4 (Pin_4), J16.7 (Pin_7), J18.A1 (GND), J18.A12 (GND), J18.B1 (GND), J18.B12 (GND), J18.S1 (SHIELD), R25.2, U5.12 (VSSA), U5.18 (VSS), U5.31 (VSS), U5.47 (VSS), U5.63 (VSS), U7.13 (GND), U7.21 (GND), U7.3 (GND), U8.3 (GND), U8.6 (GND)
- net Lid_Sensor: now also U5.8 (PC0); no longer U1.CN7_27 (PC15)
- net MOSI: no longer U1.CN7_37 (PC3)
- net PWM_SPEED: now also U5.59 (PB7); no longer U1.CN7_21 (PB7)
- net Phase_MON: no longer U1.CN10_35 (PA2)
- net READY_IN: now also J10.1 (Pin_1), U5.10 (PC2); no longer U1.CN7_2 (PC11)
- net SCL: no longer U1.CN10_3 (PB8)
- net SDA: no longer U1.CN10_5 (PB9)
- net SW_LED: now also U5.14 (PA0); no longer U1.CN7_23 (PC13)
- net aSPEED: now also R24.2
- net cRPM_METER: no longer U1.CN7_17 (PA15)
- net pBuzzer: no longer U1.CN10_4 (PC6)
- net at R6.1: now also J10.5 (Pin_5); no longer U3.14 (DIR)
- net at J3.5 (Pin_5), U3.6 (HALL_5V): no longer C2.1
- net at J3.8 (Pin_8), U3.9 (H3): no longer R11.2
- net at Q3.3 (D), R7.2: now also J10.4 (Pin_4); no longer Q2.3 (D), U3.13 (EN)
- net MISO: no longer names the net of U1.CN7_35 (PC2)
- net TEMP: no longer names the net of U1.CN10_37 (PA3)
- new net: J10.7 (Pin_7), R25.1
- new net: U7.10 (3V3OUT), U7.11 (~{RESET}), U7.20 (VCCIO)
- new net: J10.8 (Pin_8), R24.1
- new net: Q2.3 (D), U3.13 (EN)
- new net +5V: J16.5 (Pin_5)
- new net +VBUS: D5.2 (A), J18.A4 (VBUS), J18.A9 (VBUS), J18.B4 (VBUS), J18.B9 (VBUS), U7.12 (VCC)
- new net 5V_HALL: C2.1, J11.11 (Pin_11), J13.5 (Pin_5)
- new net Buzzer_PWM: U5.37 (PC6)
- new net DEBUG_SWCLK: U5.49 (PA14)
- new net DEBUG_SWDIO: U5.46 (PA13)
- new net DEBUG_SWO: U5.55 (PB3)
- new net DIG_IN1: J10.2 (Pin_2)
- new net DIG_IN2: J10.3 (Pin_3)
- new net EEPROM_WP: U5.28 (PB2)
- new net HALL_1: J11.13 (Pin_13), J13.1 (Pin_1)
- new net HALL_2: J11.15 (Pin_15), J13.2 (Pin_2)
- new net HALL_3: J11.17 (Pin_17), J13.3 (Pin_3), R11.2
- new net I2C1_SCL: U5.61 (PB8)
- new net I2C1_SDA: U5.62 (PB9)
- new net LCD_CS_DO: J17.4 (Pin_4)
- new net LCD_D0_DO: J14.10 (Pin_10), U5.39 (PC8)
- new net LCD_D1_DO: J14.9 (Pin_9), U5.40 (PC9)
- new net LCD_D2_DO: J15.6 (Pin_6), U5.51 (PC10)
- new net LCD_D3_DO: J15.5 (Pin_5), U5.52 (PC11)
- new net LCD_D4_DO: J15.4 (Pin_4), U5.53 (PC12)
- new net LCD_D5_DO: J15.3 (Pin_3), U5.2 (PC13)
- new net LCD_D6_DO: J15.2 (Pin_2), U5.3 (PC14)
- new net LCD_D7_DO: J15.1 (Pin_1), U5.4 (PC15)
- new net LCD_RD_DI: J17.1 (Pin_1)
- new net LCD_RST_DO: J17.5 (Pin_5)
- new net LCD_RS_DO: J17.3 (Pin_3)
- new net LCD_WR_DO: J17.2 (Pin_2)
- new net MCU_RST: J16.3 (Pin_3), U5.7 (NRST)
- new net Motor_1: J11.1 (Pin_1), J11.2 (Pin_2), J12.1 (Pin_1)
- new net Motor_2: J11.3 (Pin_3), J11.4 (Pin_4), J12.2 (Pin_2)
- new net Motor_3: J11.5 (Pin_5), J11.6 (Pin_6), J12.3 (Pin_3)
- new net RPM_METER_IC: U5.50 (PA15)
- new net SD_CLK: J14.5 (Pin_5)
- new net SD_CS: J14.8 (Pin_8)
- new net SD_MISO: J14.6 (Pin_6)
- new net SD_MOSI: J14.7 (Pin_7)
- new net SPI1_CLK_SD: U5.21 (PA5)
- new net SPI1_CS_SD: U5.9 (PC1)
- new net SPI1_MISO_SD: U5.22 (PA6)
- new net SPI1_MOSI_SD: U5.23 (PA7)
- new net SPI2_ADC_CS: U5.33 (PB12)
- new net SPI2_CLK: U5.34 (PB13)
- new net SPI2_MOSI: U5.11 (PC3)
- new net UART1_RX: U5.43 (PA10), U7.17 (TXD)
- new net UART1_TX: U5.42 (PA9), U7.1 (RXD)
- new net USB_DM: J18.A7 (D-), J18.B7 (D-), U7.9 (USBDM)
- new net USB_DP: J18.A6 (D+), J18.B6 (D+), U7.8 (USBDP)
- no-connect marks 24 -> 27
Other:
- note added: "Current_Limit"
- note added: "ILI9486 / ILI9488 Touch 3.5 inch TFT"
- note added: "Maxon Driver DEC 50/5 (380200)"
- note added: "Motor Connector"
- note added: "Revision History - V 1.1 [-] Change capacitor layout size to large [-] Change resistor layout size to large [-] Add zener diode to decrease heat [-] Change BJT layout pinmap [-] Change PWM reading pin to ADC pin - V 1.2 [ ] Change NPN to N-FET mosfet. [ ] Zener Diode to DC/DC Converter [ ] BEMF Block - V 1.3 [-] Change R,C,D size to SMD [-] Embedded DC/DC - v 2.0 [ ] Remove EMO [ ] Porting MCU on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"
- note added: "Speed_Set"
- note added: "TFT Display"
- note removed: "EMO_SW"
- note removed: "ENCODER_SPI"
- note removed: "ESC POWER"
- note removed: "ESC PWM"
- note removed: "Revision History - V 1.1 [-] Change capacitor layout size to large [-] Change resistor layout size to large [-] Add zener diode to decrease heat [-] Change BJT layout pinmap [-] Change PWM reading pin to ADC pin - V 1.2 [ ] Change NPN to N-FET mosfet. [ ] Zener Diode to DC/DC Converter [ ] BEMF Block - V 1.3 [-] Change R,C,D size to SMD [-] Embedded DC/DC"
- note removed: "Thermistor (NTC)"
- moved on the sheet: C10, C11, C12, C13, C14, C15, C2, C3, D1, D3, D4, J3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

Commit message: Place Arduino pinout / Drv socket
Parts:
- removed D3: MM3Z3V3T1G, Custom_Library:D_SOD-323-2, symbol Device:D_Zener
- removed J3: EH_B8B-EH-A, Connector_JST:JST_EH_B8B-EH-A_1x08_P2.50mm_Vertical, symbol Connector:Conn_01x08_Pin
- removed Q2: 2N7002, Package_TO_SOT_SMD:SOT-23, symbol Custom_Library:NMOS
- removed R10: 4.7k, Resistor_SMD:R_0603_1608Metric, symbol Device:R
- removed R2: 75k, Resistor_SMD:R_0603_1608Metric, symbol Device:R
- removed R3: 10k, Resistor_SMD:R_0603_1608Metric, symbol Device:R
- removed R4, R9: 100, Resistor_SMD:R_0603_1608Metric, symbol Device:R
- removed U1: NUCLEO-F411RE, Module:ST_NUCLEO-F401RE, symbol MCU_Module:NUCLEO-F401RE
- removed U3: 367661, Connector_Pin:MAXON_DRV, symbol Connector:MAXON_DRV
- added C16, C18: 100nF/50V, Capacitor_SMD:C_0603_1608Metric, symbol Device:C
- added C17: 2.2uF/10V, Capacitor_SMD:C_0603_1608Metric, symbol Device:C
- added R14, R26: 5.1k, Resistor_SMD:R_0603_1608Metric, symbol Device:R
- added R8: 10k, Resistor_SMD:R_0603_1608Metric, symbol Device:R
- J10: footprint Connector_PinHeader_2.54mm:PinHeader_1x08_P2.54mm_Vertical -> Connector_PinSocket_2.54mm:PinSocket_1x08_P2.54mm_Vertical
- J11: footprint Connector_PinHeader_2.54mm:PinHeader_2x09_P2.54mm_Vertical -> Connector_PinSocket_2.54mm:PinSocket_2x09_P2.54mm_Vertical
- J14: footprint (none) -> Connector_PinSocket_2.54mm:PinSocket_1x10_P2.54mm_Vertical
- J15, J16: footprint (none) -> Connector_PinSocket_2.54mm:PinSocket_1x08_P2.54mm_Vertical
- J17: footprint (none) -> Connector_PinSocket_2.54mm:PinSocket_1x06_P2.54mm_Vertical
Connections:
- net +3V3: now also C16.1
- net +VBUS: now also C18.1
- net GND: now also C16.2, C17.2, C18.2, R14.2, R26.2, R8.1
- net at J18.A5 (CC1): now also R14.1
- net at J18.B5 (CC2): now also R26.1
- net at U5.30 (VCAP1): now also C17.1
- net at U5.60 (BOOT0): now also R8.2
- no-connect marks 27 -> 4
Other:
- note added: "40Vmax"
- note added: "5A max"
- note removed: "3-40V"
- note removed: "Connectors"
- note removed: "EMR Off -> LOW EMR On -> HIGH"
- note removed: "ESC Driver hall counter"
- note removed: "Forced stop with Lid & E-STOP"
- note removed: "Motor Driver"
- moved on the sheet: J18

Commit message: finalize layout
Parts:
- added C19: 10uF/10V, Capacitor_SMD:C_0805_2012Metric, symbol Device:C
- added C20: 100nF/50V, Capacitor_SMD:C_0603_1608Metric, symbol Device:C
- added D3, D6: 150060BS55040, LED_SMD:LED_0603_1608Metric, symbol Device:LED
- added D8: MMSZ5245, Diode_SMD:D_SOD-123, symbol Custom_Library:MMSZ5245
- added J3: FTSH-105-01-L-DV-K-TR, Custom_Library:PinHeader_2x05_P1.27mm_Vertical_SMD, symbol Custom_Library:FTSH-105-01-L-DV-K-TR
- added Q4: Si7461DP, Package_SO:PowerPAK_SO-8_Single, symbol Custom_Library:Si7461DP
- added R10: 470k, Resistor_SMD:R_0603_1608Metric, symbol Device:R
- added R2, R3: 1k, Resistor_SMD:R_0603_1608Metric, symbol Device:R
- added R4: 330k, Resistor_SMD:R_0603_1608Metric, symbol Device:R
- added R9: 10, Resistor_SMD:R_0603_1608Metric, symbol Device:R
- F1: value 0679H5000-01 -> 0679H7000-01
- J1: value EH_B2B-EH-A -> Mini-Fit(5569-02A); footprint Connector_JST:JST_EH_B2B-EH-A_1x02_P2.50mm_Vertical -> Connector_Molex:Molex_Mini-Fit_Jr_5569-02A2_2x01_P4.20mm_Horizontal
- U4: footprint Package_SO:SOIC-8_5.275x5.275mm_P1.27mm -> Package_SO:SOIC-8_5.3x5.3mm_P1.27mm
Connections:
- net +E5V is gone; now on net +5V: C10.1, C11.1, C12.1, C13.1, C14.1, C15.1, C3.1, C9.1, D5.1 (K), L1.2, R19.1, U2.1 (VDD), U2.11 (VrefB), U2.13 (VrefA), U2.9 (~{SHDN}), U8.5 (EN), U8.8 (VIN)
- net ADC_CS is gone; now on net SPI2_ADC_CS: U2.3 (~{CS})
- net SCL is gone; now on net I2C1_SCL: R17.2, U4.6 (SCL)
- net SDA is gone; now on net I2C1_SDA: R16.2, U4.5 (SDA)
- net SD_CLK is gone; now on net SPI1_CLK_SD: J14.5 (Pin_5)
- net SD_CS is gone; now on net SPI1_CS_SD: J14.8 (Pin_8)
- net SD_MISO is gone; now on net SPI1_MISO_SD: J14.6 (Pin_6)
- net SD_MOSI is gone; now on net SPI1_MOSI_SD: J14.7 (Pin_7)
- net SPI2_CLK is gone; now on net SPI2_ADC_CLK: U5.34 (PB13)
- net SPI2_MOSI is gone; now on net SPI2_ADC_MOSI: U5.11 (PC3)
- net WP is gone; now on net EEPROM_WP: R18.2, U4.7 (WP)
- net cRPM_METER is gone; now on net RPM_METER_IC: R11.1
- net pBuzzer is gone; now on net Buzzer_PWM: R12.2
- net +24V: now also Q4.5 (D); no longer F1.1
- net +3V3: now also U5.1 (VBAT), C19.1, C20.1, J3.1 (Pin_1), R3.1
- net +5V: now also R2.1
- net 5V_HALL: now also J11.12 (Pin_12); no longer J11.11 (Pin_11)
- net DEBUG_SWCLK: now also J3.4 (Pin_4)
- net DEBUG_SWDIO: now also J3.2 (Pin_2)
- net DEBUG_SWO: now also J3.6 (Pin_6)
- net EEPROM_WP: now also U5.58 (PB6); no longer U5.28 (PB2)
- net GND: now also J11.13 (Pin_13), J11.15 (Pin_15), J11.17 (Pin_17), U8.9 (EP), C19.2, C20.2, D3.1 (K), D6.1 (K), J3.3 (Pin_3), J3.5 (Pin_5), J3.9 (Pin_9), R10.2; no longer J11.14 (Pin_14), J11.16 (Pin_16), J11.18 (Pin_18)
- net HALL_1: now also J11.14 (Pin_14); no longer J11.13 (Pin_13)
- net HALL_2: now also J11.16 (Pin_16); no longer J11.15 (Pin_15)
- net HALL_3: now also J11.18 (Pin_18); no longer J11.17 (Pin_17)
- net LCD_CS_DO: now also U5.44 (PA11)
- net LCD_RD_DI: now also U5.36 (PB15)
- net LCD_RST_DO: now also U5.45 (PA12)
- net LCD_RS_DO: now also U5.41 (PA8)
- net LCD_WR_DO: now also U5.38 (PC7)
- net MCU_RST: now also J3.10 (Pin_10)
- net at J5.1 (Pin_1): now also D8.2 (A), R4.2, R9.2; no longer J1.1 (Pin_1)
- net at J5.2 (Pin_2): now also R10.1; no longer F1.2
- net MOSI renamed SPI2_ADC_MOSI
- net SCK renamed SPI2_ADC_CLK
- net USB_DM renamed USB_D-
- net USB_DP renamed USB_D+
- new net: D8.1 (K), F1.1, Q4.1 (S), Q4.2 (S), Q4.3 (S), R4.1
- new net: F1.2, J1.1 (Pin_1)
- new net: D3.2 (A), R2.2
- new net: Q4.4 (G), R9.1
- new net: D6.2 (A), R3.2
Other:
- note added: "5V to 3.3V"
- note added: "DEBUG (ST-LNK)"
- note added: "MCU"
- note added: "Power_IN"
- note added: "Revision History - V 1.1 [-] Change capacitor layout size to large [-] Change resistor layout size to large [-] Add zener diode to decrease heat [-] Change BJT layout pinmap [-] Change PWM reading pin to ADC pin - V 1.2 [ ] Change NPN to N-FET mosfet. [ ] Zener Diode to DC/DC Converter [ ] BEMF Block - V 1.3 [-] Change R,C,D size to SMD [-] Embedded DC/DC - v 2.0 [-] Remove EMO [-] Porting MCU on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"
- note added: "USB to UART"
- note added: "VIN to 5V"
- note removed: "24V_Power_IN"
- note removed: "Power Distribution"
- note removed: "Revision History - V 1.1 [-] Change capacitor layout size to large [-] Change resistor layout size to large [-] Add zener diode to decrease heat [-] Change BJT layout pinmap [-] Change PWM reading pin to ADC pin - V 1.2 [ ] Change NPN to N-FET mosfet. [ ] Zener Diode to DC/DC Converter [ ] BEMF Block - V 1.3 [-] Change R,C,D size to SMD [-] Embedded DC/DC - v 2.0 [ ] Remove EMO [ ] Porting MCU on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"
- moved on the sheet: C1, C10, C11, C12, C13, C14, C15, C16, C17, C18, C2, C3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

Commit message: Output setup & layout minor fix
Parts:
- added R27: 100k, Resistor_SMD:R_0603_1608Metric, symbol Device:R
- Q4: value Si7461DP -> SI7461DP-T1-GE3
Connections:
- net GND: now also R27.1
- net Lid_Sensor: now also R27.2
Other:
- note added: "14.5mOhm @ -10Vgs Pdiss = 5A * 5A * 14.5mOhm = 0.365W"
- moved on the sheet: C1, C2, C3, C4, D1, D2, D4, D8, F1, J1, J10, J11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

Commit message: modify final output
Other:
- moved on the sheet: C10, C11, C12, C13, C14, C15, C18, C19, C20, C3, C5, C6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
